Commit message: lekiwi_description: reverse the rotation direction of the wheels to correspond to the lekiwi_hw_interface.

File: src/lekiwi_description/urdf/omni_base.xacro (robot description, xacro)
@@ -107,5 +107,5 @@
       <!-- Add PI/2 to angle so wheel +X points in rolling direction (tangent), not radial -->
       <origin xyz="0.0027 0 ${servo_offset}" rpy="0 0 ${-PI/2}"/>
-      <axis xyz="0 1 0"/>  <!-- Rotation around local Y axis (perpendicular to wheel) -->
+      <axis xyz="0 -1 0"/>  <!-- Rotation around local Y axis (perpendicular to wheel) -->
       <limit effort="10.0" velocity="10.0"/>
       <dynamics damping="0.1" friction="0.1"/>

Commit message: lekiwi_description: add LeKiwi mounted front facing camera.

File: src/lekiwi_description/urdf/omni_base.xacro (robot description, xacro)
@@ -153,3 +153,43 @@
   </joint>
   <!-- Instantiate the three omni wheels -->
+  <!-- Simulated Camera (Gazebo) -->
+  <link name="camera_link">
+    <inertial>
+      <mass value="0.1"/>
+      <origin xyz="0 0 0"/>
+      <inertia ixx="0.001" ixy="0.0" ixz="0.0" iyy="0.001" iyz="0.0" izz="0.001"/>
+    </inertial>
+    <visual>
+      <origin xyz="0 0 0" rpy="0 0 0"/>
+      <geometry>
+        <box size="0.05 0.05 0.05"/>
+      </geometry>
+      <material name="black"/>
+    </visual>
+  </link>
+  <joint name="camera_joint" type="fixed">
+    <parent link="base_footprint"/>
+    <child link="camera_link"/>
+    <origin xyz="0.09 0 0.065" rpy="0 0 0"/>
+  </joint>
+  <gazebo reference="camera_link">
+    <sensor type="camera" name="camera_link">
+      <always_on>true</always_on>
+      <update_rate>30.0</update_rate>
+      <visualize>true</visualize>
+      <camera>
+        <horizontal_fov>1.3962634</horizontal_fov>
+        <image>
+          <width>640</width>
+          <height>480</height>
+          <format>R8G8B8</format>
+        </image>
+        <clip>
+          <near>0.1</near>
+          <far>100</far>
+        </clip>
+      </camera>
+      <topic>lekiwi_front_camera/image</topic>
+    </sensor>
+  </gazebo>
 </robot>
